File: RF-fix-code-2-relay-hw/RF-fix-code-2-relay-hw.sch (KiCad schematic (older format))
At the start: 19 parts

Commit message: complete rf-fix-code-2-relay-hw
Parts:
- removed C? (x2): C, Capacitors_SMD:C_0805_HandSoldering, symbol C
- removed D? (x3): D_ALT, symbol D_ALT
- removed SW?: SW-8-3-State, nhantt-kicad-lib:SW-8-3-state, symbol SW-8-3-State
- added C1, C11, C2, C4, C6, C7, C9: 100nF, Capacitors_ThroughHole:C_Disc_D3_P2.5, symbol C
- added C10, C8: 2kV, nhantt-kicad-lib:C_103_2KV, symbol C
- added C3, C5: CP1, Capacitors_ThroughHole:C_Radial_D8_L13_P3.8, symbol CP1
- added D2: D_ALT, Diodes_ThroughHole:Diode_DO-201AD_Horizontal_RM15, symbol D_ALT
- added D4, D5, D6, D7, D8: D_ALT, Diodes_ThroughHole:Diode_DO-41_SOD81_Horizontal_RM10, symbol D_ALT
- added J2, J3, J4: CONN_01X02, nhantt-kicad-lib:Domino-5.08mm_2pol, symbol CONN_01X02
- added M2: RF315, nhantt-kicad-lib:RF_YKTR-5S, symbol RF315
- added Q1, Q2: 2SC1815, TO_SOT_Packages_THT:TO-92_Molded_Wide_Oval, symbol 2SC1815
- added R10, R12: 10k, Resistors_ThroughHole:Resistor_Horizontal_RM10mm, symbol R
- added R11: 330, Resistors_ThroughHole:Resistor_Horizontal_RM10mm, symbol R
- added R13, R9: 2.2k, Resistors_ThroughHole:Resistor_Horizontal_RM10mm, symbol R
- added R4: R, Resistors_ThroughHole:Resistor_Horizontal_RM10mm, symbol R
- added RL1, RL2: G5Q-1, nhantt-kicad-lib:Relay_SRD-SONGLE, symbol G5Q-1
- added SW1: SW-8-3-State, nhantt-kicad-lib:SW-8-3-state, symbol SW-8-3-State
- added U2: LM7805CT, TO_SOT_Packages_THT:TO-92_Molded_Wide_Oval, symbol LM7805CT
- D1: renamed from D?; footprint (none) -> LEDs:LED-5MM
- D3: renamed from D?; footprint (none) -> Diodes_ThroughHole:Diode_DO-41_SOD81_Horizontal_RM10
- J1: renamed from J?; footprint (none) -> nhantt-kicad-lib:PAD_Rec
- R1, R2, R7, R8: renamed from R?; footprint (none) -> Resistors_ThroughHole:Resistor_Horizontal_RM10mm
- R5, R6: renamed from R?; footprint (none) -> Resistors_SMD:R_0805_HandSoldering
- U3: renamed from U?; footprint (none) -> Housings_DIP:DIP-14_W7.62mm_LongPads
- gave numbers to parts that had none: 2
Connections:
- net OUTA is gone; now on net OUT2: R7.2
- net VDD is gone; now on net VCC: U3.14 (VDD), U3.14 (VDD)
- net VSS is gone; now on net GND: U3.7 (VSS), U3.7 (VSS)
- net GND: now also C1.2, C11.2, C2.2, C3.2, C4.2, C5.2, C6.2, C7.2, J2.1 (P1), M2.4 (GND), Q1.1 (E), Q2.1 (E), R10.1, R12.1, SW1.8 (B), U2.2 (GND)
- net OUT1: now also D4.1 (K), R11.2
- net OUT2: now also D5.1 (K), D6.1 (K)
- net VCC: now also C1.1, C11.1, C2.1, C5.1, C6.1, C7.1, C9.1, M2.1 (VCC), SW1.1 (A), U2.3 (OUT)
- net reset: now also C9.2, R10.2
- net at U1.1 (A0): now also SW1.16 (8)
- net at U1.10 (D0): now also D6.2 (A)
- net at U1.11 (D1): now also D5.2 (A)
- net at U1.12 (D2): now also D4.2 (A)
- net data: now reaches M1.2 (OUT), U1.14 (DIN)
- net data: now also M2.2 (DATA), M2.3 (DATA)
- net at U1.2 (A1): now also SW1.15 (7)
- net at U1.3 (A2): now also SW1.14 (6)
- net at U1.4 (A3): now also SW1.13 (5)
- net at U1.5 (A4): now also SW1.12 (4)
- net at U1.6 (A4): now also SW1.11 (3)
- net at U1.7 (A6): now also SW1.10 (2)
- net at U1.8 (A7): now also SW1.9 (1)
- net at U3.1 (Q): now also R9.1
- net at U3.11 (Cp): now also R11.1, R12.2
- net at U3.13 (Q): now also R13.1
- new net: D7.2 (A), Q1.2 (C), RL1.2
- new net: C8.1, J3.1 (P1), RL1.3
- new net: C8.2, J3.2 (P2), RL1.1
- new net: C3.1, C4.1, R4.2, U2.1 (IN)
- new net: Q1.3 (B), R9.2
- new net: D8.2 (A), Q2.2 (C), RL2.2
- new net: C10.1, J4.1 (P1), RL2.3
- new net: C10.2, J4.2 (P2), RL2.1
- new net: Q2.3 (B), R13.2
- new net: D2.2 (A), J2.2 (P2)
- new net +12V: D2.1 (K), D7.1 (K), D8.1 (K), R4.1, RL1.5, RL2.5
- no-connect marks 0 -> 2
Other:
- moved on the sheet: R7, R8, U3A, U3B
